Commit message: import logiee-s-tc urdf and mesh

File: logiee-s-tc_description/urdf/vehicle.xacro (robot description, xacro)
@@ -2,11 +2,11 @@
 <robot xmlns:xacro="http://ros.org/wiki/xacro">
   <!-- load parameter -->
-  <xacro:property name="vehicle_info" value="${xacro.load_yaml('$(find sample_vehicle_description)/config/vehicle_info.param.yaml')}"/>
+  <xacro:property name="vehicle_info" value="${load_yaml('$(find logiee_s-tc_description)/config/vehicle_info.param.yaml')}"/>
   <!-- vehicle body -->
   <link name="base_link">
     <visual>
-      <origin xyz="${vehicle_info['/**']['ros__parameters']['wheel_base']/2.0} 0 0" rpy="${pi/2.0} 0 ${pi}"/>
+      <origin xyz="0 0 0" rpy="0 0 0"/>
       <geometry>
-        <mesh filename="package://sample_vehicle_description/mesh/lexus.dae" scale="1 1 1"/>
+        <mesh filename="package://logiee_s-tc_description/mesh/LogieeS-TC.dae" scale="1 1 1"/>
       </geometry>
     </visual>

Commit message: apply setting

File: logiee-s-tc_description/urdf/vehicle.xacro (robot description, xacro)
@@ -2,11 +2,14 @@
 <robot xmlns:xacro="http://ros.org/wiki/xacro">
   <!-- load parameter -->
-  <xacro:property name="vehicle_info" value="${load_yaml('$(find logiee_s-tc_description)/config/vehicle_info.param.yaml')}"/>
+  <xacro:property name="vehicle_info" value="${xacro.load_yaml('$(find logiee_s-tc_description)/config/vehicle_info.param.yaml')}"/>
   <!-- vehicle body -->
   <link name="base_link">
     <visual>
       <origin xyz="0 0 0" rpy="0 0 0"/>
+      <!-- <geometry>
+        <mesh filename="package://logiee_s-tc_description/mesh/LogieeS-TC.dae" scale="1 1 1"/>
+      </geometry> -->
       <geometry>
-        <mesh filename="package://logiee_s-tc_description/mesh/LogieeS-TC.dae" scale="1 1 1"/>
+          <cylinder length="0.6" radius="0.4"/>
       </geometry>
     </visual>
